Commit message: date_22_11_13

File: install/tribot/share/tribot/urdf/tribot_base.xacro (robot description, xacro)
@@ -41,5 +41,5 @@
             <geometry>
                 <mesh
-                filename="package://tribot_description/meshes/base_link.STL" />
+                filename="package://tribot/meshes/base_link.STL" />
             </geometry>
             <material
@@ -55,5 +55,5 @@
             <geometry>
                 <mesh
-                filename="package://tribot_description/meshes/base_link.STL" />
+                filename="package://tribot/meshes/base_link.STL" />
             </geometry>
             </collision>

File: install/tribot/share/tribot/urdf/tribot_camera.xacro (robot description, xacro)
@@ -24,5 +24,5 @@
                 <geometry>
                     <mesh
-                    filename="package://tribot_description/meshes/camera_link.STL" />
+                    filename="package://tribot/meshes/camera_link.STL" />
                 </geometry>
                 <material
@@ -38,5 +38,5 @@
                 <geometry>
                     <mesh
-                    filename="package://tribot_description/meshes/camera_link.STL" />
+                    filename="package://tribot/meshes/camera_link.STL" />
                 </geometry>
             </collision>

File: install/tribot/share/tribot/urdf/tribot_description.urdf (robot description, URDF)
Before this commit: robot tribot_description, 6 links, 5 joints
Links:
- link base_link: geometry collision mesh filename=package://tribot/meshes/base_link.STL; visual mesh filename=package://tribot/meshes/base_link.STL
- link camera_link: geometry collision mesh filename=package://tribot/meshes/camera_link.STL; visual mesh filename=package://tribot/meshes/camera_link.STL
- link lidar_link: geometry collision mesh filename=package://tribot/meshes/lidar_link.STL; visual mesh filename=package://tribot/meshes/lidar_link.STL
- link wheel1_link: geometry collision mesh filename=package://tribot/meshes/wheel1_link.STL; visual mesh filename=package://tribot/meshes/wheel1_link.STL
- link wheel2_link: geometry collision mesh filename=package://tribot/meshes/wheel2_link.STL; visual mesh filename=package://tribot/meshes/wheel2_link.STL
- link wheel3_link: geometry collision mesh filename=package://tribot/meshes/wheel3_link.STL; visual mesh filename=package://tribot/meshes/wheel3_link.STL

File: install/tribot/share/tribot/urdf/tribot_gazebo.xacro (robot description, xacro)
@@ -2,7 +2,7 @@
 <robot name="tribot" xmlns:xacro="http://www.ros.org/wiki/xacro">
     <xacro:property name="M_PI" value="3.1415926"/>
-    <xacro:include filename="$(find tribot_description)/urdf/tribot_base.xacro" />
+    <xacro:include filename="$(find tribot)/urdf/tribot_base.xacro" />
     <xacro:tribot_base/>
-    <xacro:include filename="$(find tribot_description)/urdf/tribot_wheel.xacro" />
+    <xacro:include filename="$(find tribot)/urdf/tribot_wheel.xacro" />
       <link
         name="wheel1_link">
@@ -27,5 +27,5 @@
           <geometry>
             <mesh
-              filename="package://tribot_description/meshes/wheel1_link.STL" />
+              filename="package://tribot/meshes/wheel1_link.STL" />
           </geometry>
           <material
@@ -41,5 +41,5 @@
           <geometry>
             <mesh
-              filename="package://tribot_description/meshes/wheel1_link.STL" />
+              filename="package://tribot/meshes/wheel1_link.STL" />
           </geometry>
         </collision>
@@ -59,5 +59,5 @@
       </joint>
     <xacro:tribot_wheel prefix="wheel1"/>
-    <xacro:include filename="$(find tribot_description)/urdf/tribot_wheel.xacro" />
+    <xacro:include filename="$(find tribot)/urdf/tribot_wheel.xacro" />
       <link
         name="wheel2_link">
@@ -82,5 +82,5 @@
           <geometry>
             <mesh
-              filename="package://tribot_description/meshes/wheel2_link.STL" />
+              filename="package://tribot/meshes/wheel2_link.STL" />
           </geometry>
           <material
@@ -96,5 +96,5 @@
           <geometry>
             <mesh
-              filename="package://tribot_description/meshes/wheel2_link.STL" />
+              filename="package://tribot/meshes/wheel2_link.STL" />
           </geometry>
         </collision>
@@ -114,5 +114,5 @@
       </joint>
     <xacro:tribot_wheel prefix="wheel2"/>
-    <xacro:include filename="$(find tribot_description)/urdf/tribot_wheel.xacro" />
+    <xacro:include filename="$(find tribot)/urdf/tribot_wheel.xacro" />
       <link
         name="wheel3_link">
@@ -137,5 +137,5 @@
           <geometry>
             <mesh
-              filename="package://tribot_description/meshes/wheel3_link.STL" />
+              filename="package://tribot/meshes/wheel3_link.STL" />
           </geometry>
           <material
@@ -151,5 +151,5 @@
           <geometry>
             <mesh
-              filename="package://tribot_description/meshes/wheel3_link.STL" />
+              filename="package://tribot/meshes/wheel3_link.STL" />
           </geometry>
         </collision>
@@ -169,5 +169,5 @@
       </joint>
     <xacro:tribot_wheel prefix="wheel3"/>
-    <xacro:include filename="$(find tribot_description)/urdf/tribot_lidar.xacro" />
+    <xacro:include filename="$(find tribot)/urdf/tribot_lidar.xacro" />
       <joint
         name="lidar_joint"
@@ -184,5 +184,5 @@
       </joint>
     <xacro:tribot_lidar/>
-    <xacro:include filename="$(find tribot_description)/urdf/tribot_camera.xacro" />
+    <xacro:include filename="$(find tribot)/urdf/tribot_camera.xacro" />
       <joint
         name="camera_joint"

File: install/tribot/share/tribot/urdf/tribot_lidar.xacro (robot description, xacro)
@@ -25,5 +25,5 @@
             <geometry>
                 <mesh
-                filename="package://tribot_description/meshes/lidar_link.STL" />
+                filename="package://tribot/meshes/lidar_link.STL" />
             </geometry>
             <material
@@ -39,5 +39,5 @@
             <geometry>
                 <mesh
-                filename="package://tribot_description/meshes/lidar_link.STL" />
+                filename="package://tribot/meshes/lidar_link.STL" />
             </geometry>
             </collision>
